File: KiCAD Repo/Power_Elec_Project-2025-01-26_221946/GATE_DRIVER.kicad_sch (KiCad schematic)
At the start: 19 parts, among them U3 UCC5304DWVR, U4 TMV 0512SHI

Commit message: PCB
Parts:
- D1: Part Number (none) -> US2AA
Changed lines of the file:
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@@
+			)
+		)
+		(property "Part Number" "US2AA"
+			(at 200.66 127 0)
+			(effects
+				(font
+					(size 1.27 1.27)
+				)
+				(hide yes)
 			)
 		)
