File: KiCAD Repo/Power_Elec_Project-2025-01-26_221946/Power_Elec_Project.kicad_pcb (KiCad board)
At the start: 2 copper layers, 131.5 x 128.2 mm, 56 parts, among them J1 RED, J2 RED, J3 RED, J4 Black, J5 Black, Q1 IRF540N, U2 LAUNCHXL-F28379D, U3 UCC5304DWVR, U4 TMV 0512SHI, U5 AMC1300DWVR

Commit message: Added Name and logo on silkscreen
Parts:
- added G***: LOGO, LOGO, F.Cu at (102.0, 52.0)
Other:
- board text added: "ELEC-4450 M.Nguyen B.Patel S.Dupuis"
